Commit message: Split urdf to multiple xacro and include in final xacro

File: src/castor_wheel_robot_description/urdf/castor_wheel_robot.urdf.xacro (robot description, xacro)
@@ -1,90 +1,7 @@
 <?xml version="1.0"?>
 <robot name="Castor Wheel Robot" xmlns:xacro="http://www.ros.org/wiki/xacro">
-    <!-- Material Blue -->
-    <material name="blue">
-        <color rgba="0 0 1 1"/>
-    </material>
-    <!-- Material Red -->
-    <material name="red">
-        <color rgba="1 0 0 1"/>
-    </material>
-    <!-- Material Green -->
-    <material name="green">
-        <color rgba="0 1 0 1"/>
-    </material>
-    <!-- Macros -->
-    <xacro:property name="base_length" value="0.6"/>
-    <xacro:property name="base_width" value="0.4"/>
-    <xacro:property name="base_height" value="0.2"/>
-    <xacro:property name="wheel_radius" value="0.1"/>
-    <xacro:property name="wheel_length" value="0.05"/>
-    <!-- Empty footprint link -->
-    <link name="base_footprint">
-    </link>
-    <!-- Robot base link -->
-    <link name="base_link">
-        <visual>
-            <geometry>
-                <box size="${base_length} ${base_width} ${base_height}"/>
-            </geometry>
-            <material name="blue"/>
-            <origin xyz="0 0 ${base_height/2}" rpy="0 0 0"/>
-        </visual>
-    </link>
-    <!-- Joint between base_footprint and base -->
-    <joint name="base_footprint_base_link_joint" type="fixed">
-        <parent link="base_footprint"/>
-        <child link="base_link"/>
-        <origin xyz="0 0 ${wheel_radius}" rpy="0 0 0"/>
-    </joint>
-    <!-- Left Wheel Link -->
-    <link name="left_wheel">
-        <visual>
-            <geometry>
-                <cylinder radius="${wheel_radius}" length="${wheel_length}"/>
-            </geometry>
-            <material name="green"/>
-            <origin xyz="0 0 0" rpy="0 0 0"/>
-        </visual>
-    </link>
-    <!-- Joint between base and left wheel -->
-    <joint name="base_link_left_wheel_joint" type="continuous">
-        <parent link="base_link"/>
-        <child link="left_wheel"/>
-        <origin xyz="${-base_length/4} ${(base_width/2) + (wheel_length/2)} 0" rpy="${pi/2} 0 0"/>
-        <axis xyz="0 0 1"/>
-    </joint>
-    <!-- Right Wheel Link -->
-    <link name="right_wheel">
-        <visual>
-            <geometry>
-                <cylinder radius="${wheel_radius}" length="${wheel_length}"/>
-            </geometry>
-            <material name="green"/>
-            <origin xyz="0 0 0" rpy="0 0 0"/>
-        </visual>
-    </link>
-    <!-- Joint between base and right wheel -->
-    <joint name="base_link_right_wheel_joint" type="continuous">
-        <parent link="base_link"/>
-        <child link="right_wheel"/>
-        <origin xyz="${-base_length/4} ${-((base_width/2) + (wheel_length/2))} 0" rpy="${pi/2} 0 0"/>
-        <axis xyz="0 0 1"/>
-    </joint>
-    <!-- Castor Wheel Link -->
-    <link name="castor_wheel">
-        <visual>
-            <geometry>
-                <sphere radius="${wheel_radius/2}"/>
-            </geometry>
-            <material name="green"/>
-            <origin xyz="0 0 0" rpy="0 0 0"/>
-        </visual>
-    </link>
-    <!-- Joint between base and castor wheel -->
-    <joint name="base_link_castor_wheel_joint" type="fixed">
-        <parent link="base_link"/>
-        <child link="castor_wheel"/>
-        <origin xyz="${base_length/3} 0 ${-wheel_radius/2}" rpy="0 0 0"/>
-    </joint>
+    <!-- Common Properties File -->
+    <xacro:include filename="common_properties.xacro"/>
+    <!-- Mobile Base File -->
+    <xacro:include filename="mobile_base.xacro"/>
 </robot>
