Commit message: Added collision tags

File: src/castor_wheel_robot_description/urdf/mobile_base.xacro (robot description, xacro)
@@ -19,4 +19,10 @@
             <origin xyz="0 0 ${base_height/2}" rpy="0 0 0"/>
         </visual>
+        <collision>
+            <geometry>
+                <box size="${base_length} ${base_width} ${base_height}"/>
+            </geometry>
+            <origin xyz="0 0 ${base_height/2}" rpy="0 0 0"/>
+        </collision>
         <xacro:box_inertia m="5.0" l="${base_length}" w="${base_width}" h="${base_height}" xyz="0 0 ${base_height/2}" rpy="0 0 0"/>
     </link>
@@ -36,4 +42,10 @@
             <origin xyz="0 0 0" rpy="0 0 0"/>
         </visual>
+        <collision>
+            <geometry>
+                <cylinder radius="${wheel_radius}" length="${wheel_length}"/>
+            </geometry>
+            <origin xyz="0 0 0" rpy="0 0 0"/>
+        </collision>
         <xacro:cylinder_inertia m="1.0" r="${wheel_radius}" l="${wheel_length}" xyz="0 0 0" rpy="0 0 0"/>
     </link>
@@ -54,4 +66,10 @@
             <origin xyz="0 0 0" rpy="0 0 0"/>
         </visual>
+        <collision>
+            <geometry>
+                <cylinder radius="${wheel_radius}" length="${wheel_length}"/>
+            </geometry>
+            <origin xyz="0 0 0" rpy="0 0 0"/>
+        </collision>
         <xacro:cylinder_inertia m="1.0" r="${wheel_radius}" l="${wheel_length}" xyz="0 0 0" rpy="0 0 0"/>
     </link>
@@ -72,4 +90,10 @@
             <origin xyz="0 0 0" rpy="0 0 0"/>
         </visual>
+        <collision>
+            <geometry>
+                <sphere radius="${wheel_radius/2}"/>
+            </geometry>
+            <origin xyz="0 0 0" rpy="0 0 0"/>
+        </collision>
         <xacro:sphere_inertia m="0.5" r="${wheel_radius/2}" xyz="0 0 0" rpy="0 0 0"/>
     </link>

Commit message: Fixed the issue of robot driving backwards due to origin of wheels

File: src/castor_wheel_robot_description/urdf/mobile_base.xacro (robot description, xacro)
@@ -40,5 +40,5 @@
             </geometry>
             <material name="green"/>
-            <origin xyz="0 0 0" rpy="0 0 0"/>
+            <origin xyz="0 0 0" rpy="${pi/2} 0 0"/>
         </visual>
         <collision>
@@ -46,7 +46,7 @@
                 <cylinder radius="${wheel_radius}" length="${wheel_length}"/>
             </geometry>
-            <origin xyz="0 0 0" rpy="0 0 0"/>
+            <origin xyz="0 0 0" rpy="${pi/2} 0 0"/>
         </collision>
-        <xacro:cylinder_inertia m="1.0" r="${3*wheel_radius}" l="${3*wheel_length}" xyz="0 0 0" rpy="0 0 0"/>
+        <xacro:cylinder_inertia m="1.0" r="${3*wheel_radius}" l="${3*wheel_length}" xyz="0 0 0" rpy="${pi/2} 0 0"/>
     </link>
     <!-- Joint between base and left wheel -->
@@ -54,6 +54,6 @@
         <parent link="base_link"/>
         <child link="left_wheel"/>
-        <origin xyz="${-base_length/4} ${(base_width/2) + (wheel_length/2)} 0" rpy="${pi/2} 0 0"/>
-        <axis xyz="0 0 1"/>
+        <origin xyz="${-base_length/4} ${(base_width/2) + (wheel_length/2)} 0" rpy="0 0 0"/>
+        <axis xyz="0 1 0"/>
     </joint>
     <!-- Right Wheel Link -->
@@ -64,5 +64,5 @@
             </geometry>
             <material name="green"/>
-            <origin xyz="0 0 0" rpy="0 0 0"/>
+            <origin xyz="0 0 0" rpy="${pi/2} 0 0"/>
         </visual>
         <collision>
@@ -70,7 +70,7 @@
                 <cylinder radius="${wheel_radius}" length="${wheel_length}"/>
             </geometry>
-            <origin xyz="0 0 0" rpy="0 0 0"/>
+            <origin xyz="0 0 0" rpy="${pi/2} 0 0"/>
         </collision>
-        <xacro:cylinder_inertia m="1.0" r="${3*wheel_radius}" l="${3*wheel_length}" xyz="0 0 0" rpy="0 0 0"/>
+        <xacro:cylinder_inertia m="1.0" r="${3*wheel_radius}" l="${3*wheel_length}" xyz="0 0 0" rpy="${pi/2} 0 0"/>
     </link>
     <!-- Joint between base and right wheel -->
@@ -78,6 +78,6 @@
         <parent link="base_link"/>
         <child link="right_wheel"/>
-        <origin xyz="${-base_length/4} ${-((base_width/2) + (wheel_length/2))} 0" rpy="${pi/2} 0 0"/>
-        <axis xyz="0 0 1"/>
+        <origin xyz="${-base_length/4} ${-((base_width/2) + (wheel_length/2))} 0" rpy="0 0 0"/>
+        <axis xyz="0 1 0"/>
     </joint>
     <!-- Castor Wheel Link -->
