Commit message: Inertial tags added for all components

File: src/castor_wheel_robot_description/urdf/common_properties.xacro (robot description, xacro)
@@ -13,3 +13,28 @@
         <color rgba="0 1 0 1"/>
     </material>
+    <!-- Inertial Tags -->
+    <!-- Box Inertia -->
+    <xacro:macro name="box_inertia" params="m l w h xyz rpy">
+        <inertial>
+            <origin xyz="${xyz}" rpy="${rpy}"/>
+            <mass value="${m}"/>
+            <inertia ixx="${(m/12)*(h*h+l*l)}" ixy="0.0" ixz="0.0" iyy="${(m/12)*(h*h+w*w)}" iyz="0.0" izz="${(m/12)*(w*w+l*l)}"/>
+        </inertial>
+    </xacro:macro>
+    <!-- Cylinder Inertia -->
+    <xacro:macro name="cylinder_inertia" params="m r l xyz rpy">
+        <inertial>
+            <origin xyz="${xyz}" rpy="${rpy}"/>
+            <mass value="${m}"/>
+            <inertia ixx="${(m/12)*((3*r*r)+(l*l))}" ixy="0.0" ixz="0.0" iyy="${(m/12)*((3*r*r)+(l*l))}" iyz="0.0" izz="${(m/2)*r*r}"/>
+        </inertial>
+    </xacro:macro>
+    <!-- Sphere Inertia -->
+    <xacro:macro name="sphere_inertia" params="m r xyz rpy">
+        <inertial>
+            <origin xyz="${xyz}" rpy="${rpy}"/>
+            <mass value="${m}"/>
+            <inertia ixx="${2/5*m*r*r}" ixy="0.0" ixz="0.0" iyy="${2/5*m*r*r}" iyz="0.0" izz="${2/5*m*r*r}"/>
+        </inertial>
+    </xacro:macro>
 </robot>

File: src/castor_wheel_robot_description/urdf/mobile_base.xacro (robot description, xacro)
@@ -19,4 +19,5 @@
             <origin xyz="0 0 ${base_height/2}" rpy="0 0 0"/>
         </visual>
+        <xacro:box_inertia m="5.0" l="${base_length}" w="${base_width}" h="${base_height}" xyz="0 0 ${base_height/2}" rpy="0 0 0"/>
     </link>
     <!-- Joint between base_footprint and base -->
@@ -35,4 +36,5 @@
             <origin xyz="0 0 0" rpy="0 0 0"/>
         </visual>
+        <xacro:cylinder_inertia m="1.0" r="${wheel_radius}" l="${wheel_length}" xyz="0 0 0" rpy="0 0 0"/>
     </link>
     <!-- Joint between base and left wheel -->
@@ -52,4 +54,5 @@
             <origin xyz="0 0 0" rpy="0 0 0"/>
         </visual>
+        <xacro:cylinder_inertia m="1.0" r="${wheel_radius}" l="${wheel_length}" xyz="0 0 0" rpy="0 0 0"/>
     </link>
     <!-- Joint between base and right wheel -->
@@ -69,4 +72,5 @@
             <origin xyz="0 0 0" rpy="0 0 0"/>
         </visual>
+        <xacro:sphere_inertia m="0.5" r="${wheel_radius/2}" xyz="0 0 0" rpy="0 0 0"/>
     </link>
     <!-- Joint between base and castor wheel -->

Commit message: Added Arm in rviz

File: src/castor_wheel_robot_description/urdf/common_properties.xacro (robot description, xacro)
@@ -12,4 +12,12 @@
     <material name="green">
         <color rgba="0 1 0 1"/>
+    </material>
+    <!-- Material Orange -->
+    <material name="orange">
+        <color rgba="1 0.5 0 1"/>
+    </material>
+    <!-- Material Yellow -->
+    <material name="yellow">
+        <color rgba="1 1 0 1"/>
     </material>
     <!-- Inertial Tags -->
