Commit message: Arm plugins and gazebo properties added for standalone

File: src/castor_wheel_robot_description/urdf/arm.xacro (robot description, xacro)
@@ -14,6 +14,13 @@
             </geometry>
             <material name="orange"/>
-            <origin xyz="0 0 0" rpy="0 0 0"/>
+            <origin xyz="0 0 ${arm_base_height/2}" rpy="0 0 0"/>
         </visual>
+        <collision>
+            <geometry>
+                <box size="${arm_base_length} ${arm_base_width} ${arm_base_height}"/>
+            </geometry>
+            <origin xyz="0 0 ${arm_base_height/2}" rpy="0 0 0"/>
+        </collision>
+        <xacro:box_inertia m="0.5" l="${arm_base_length}" w="${arm_base_width}" h="${arm_base_height}" xyz="0 0 ${arm_base_height}" rpy="0 0 0"/>
     </link>
     <!-- Forearm link -->
@@ -26,7 +33,14 @@
             <origin xyz="0 0 ${arm_length/2}" rpy="0 0 0"/>
         </visual>
+        <collision>
+            <geometry>
+                <cylinder radius="${arm_radius}" length="${arm_length}"/>
+            </geometry>
+            <origin xyz="0 0 ${arm_length/2}" rpy="0 0 0"/>
+        </collision>
+        <xacro:cylinder_inertia m="0.3" r="${arm_radius}" l="${arm_length}" xyz="0 0 ${arm_length/2}" rpy="0 0 0"/>
     </link>
     <!-- Joint between arm_base_link and forearm_link -->
-    <joint name="arm_base_link_forearm_link_joint" type="revolute">
+    <joint name="arm_base_forearm_joint" type="revolute">
         <parent link="arm_base_link"/>
         <child link="forearm_link"/>
@@ -45,7 +59,14 @@
             <origin xyz="0 0 ${arm_length/2}" rpy="0 0 0"/>
         </visual>
+        <collision>
+            <geometry>
+                <cylinder radius="${arm_radius}" length="${arm_length}"/>
+            </geometry>
+            <origin xyz="0 0 ${arm_length/2}" rpy="0 0 0"/>
+        </collision>
+        <xacro:cylinder_inertia m="0.3" r="${arm_radius}" l="${arm_length}" xyz="0 0 ${arm_length/2}" rpy="0 0 0"/>
     </link>
     <!-- Joint between forearm_link and hand_link -->
-    <joint name="forearm_link_hand_link_joint" type="revolute">
+    <joint name="forearm_hand_joint" type="revolute">
         <parent link="forearm_link"/>
         <child link="hand_link"/>

File: src/castor_wheel_robot_description/urdf/standalone_arm.urdf.xacro (robot description, xacro)
@@ -5,3 +5,5 @@
     <!-- Arm File -->
     <xacro:include filename="arm.xacro"/>
+    <!-- Gazebo Properties -->
+    <xacro:include filename="arm_gazebo.xacro"/>
 </robot>
